Commit message: Add gripper collision in urdf

File: jetcobot_description/urdf/mycobot_280_m5/mycobot_280m5_with_gripper_parallel.urdf (robot description, URDF)
Before this commit: robot firefighter, 16 links, 15 joints
Links:
- link gripper_left1: geometry collision box size=0.015 0.06 0.02; visual mesh filename=package://jetcobot_description/urdf/mycobot_280_m5/gripper_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
- link gripper_right1: geometry collision box size=0.015 0.06 0.02; visual mesh filename=package://jetcobot_description/urdf/mycobot_280_m5/gripper_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

Commit message: Add 'TCP' link at jetcobot

File: jetcobot_description/urdf/mycobot_280_m5/mycobot_280m5_with_gripper_parallel.urdf (robot description, URDF)
Before this commit: robot firefighter, 16 links, 15 joints
Links:
- added link TCP; visual box size=0.01 0.01 0.01
Joints:
- added joint gripper_base_to_TCP: type fixed, parent gripper_base, child TCP, origin xyz=0 0.07 0 rpy=-1.5708 3.1416 0

Commit message: Adjusts jetcocam position in mycobot URDF
Corrects the position and orientation of the jetcocam within the mycobot URDF for improved visual alignment and collision accuracy.

Specifically, modifies the origin of both the visual and collision elements of the "jetcocam" link, and adjusts the joint connecting the gripper base to the jetcocam.

File: jetcobot_description/urdf/mycobot_280_m5/mycobot_280m5_with_gripper_parallel.urdf (robot description, URDF)
Before this commit: robot firefighter, 17 links, 16 joints
Links:
- link jetcocam: geometry collision box size=0.04 0.05 0.015; visual box size=0.04 0.05 0.015
Joints:
- joint gripper_base_to_jetcocam: origin xyz=0 0 -0.048 rpy=-1.5708 3.1416 0 -> xyz=0 -0.01 -0.048 rpy=-1.5708 3.1416 0
