Commit message: Change jetcobot URDF's TCP joint position

File: jetcobot_description/urdf/jetcobot.urdf (robot description, URDF)
Before this commit: robot jetcobot, 11 links, 10 joints
Joints:
- joint TCP_joint: origin xyz=0.05 0 0.02 rpy=-1.5707963 0 -1.5707963 -> xyz=0.05 0 0.0177 rpy=-1.5707963 0 -1.5707963

Commit message: Edit joint lilmit

File: jetcobot_description/urdf/jetcobot.urdf (robot description, URDF)
Before this commit: robot jetcobot, 11 links, 10 joints
Joints:
- joint 1_Joint: limit lower=-3.14 upper=3.14159 effort=0 velocity=0 -> lower=-3.14 upper=3.14 effort=0 velocity=0
- joint 2_Joint: limit lower=-2.9322 upper=2.9322 effort=0 velocity=0 -> lower=-2.9 upper=2.9 effort=0 velocity=0
- joint 3_Joint: limit lower=-2.3562 upper=2.3562 effort=0 velocity=0 -> lower=-2.3 upper=2.3 effort=0 velocity=0
- joint 4_Joint: limit lower=-2.618 upper=2.618 effort=0 velocity=0 -> lower=-2.6 upper=2.6 effort=0 velocity=0
- joint 5_Joint: limit lower=-2.5307 upper=2.5307 effort=0 velocity=0 -> lower=-2.5 upper=2.5 effort=0 velocity=0
- joint 6_Joint: limit lower=-2.8798 upper=2.8798 effort=0 velocity=0 -> lower=-2.84 upper=2.84 effort=0 velocity=0

Commit message: Add new camera 'ov3360'

File: jetcobot_description/urdf/jetcobot.urdf (robot description, URDF)
Before this commit: robot jetcobot, 11 links, 10 joints
Links:
- added link ov3360
Joints:
- added joint ov3360_joint: type fixed, parent jetcocam, child ov3360, origin xyz=0.0 0.0 0.0 rpy=0 0 3.141592

Commit message: initial commit of hybrid planning

File: jetcobot_description/urdf/jetcobot.urdf (robot description, URDF)
Before this commit: robot jetcobot, 12 links, 11 joints
Joints:
- joint 1_Joint: limit lower=-3.14 upper=3.14 effort=0 velocity=0 -> lower=-3.14 upper=3.14 effort=50.0 velocity=2.5
- joint 2_Joint: limit lower=-2.9 upper=2.9 effort=0 velocity=0 -> lower=-2.9 upper=2.9 effort=40.0 velocity=2.5
- joint 3_Joint: limit lower=-2.3 upper=2.3 effort=0 velocity=0 -> lower=-2.3 upper=2.3 effort=30.0 velocity=2.5
- joint 4_Joint: limit lower=-2.6 upper=2.6 effort=0 velocity=0 -> lower=-2.6 upper=2.6 effort=20.0 velocity=2.5
- joint 5_Joint: limit lower=-2.5 upper=2.5 effort=0 velocity=0 -> lower=-2.5 upper=2.5 effort=15.0 velocity=2.5
- joint 6_Joint: limit lower=-2.84 upper=2.84 effort=0 velocity=0 -> lower=-2.84 upper=2.84 effort=10.0 velocity=2.5
