Commit message: Add URDF and change name of stl files

File: jetcobot_description/urdf/jetcobot_display.urdf (robot description, URDF)
Before this commit: robot jetcobot, 16 links, 15 joints
Links:
- link 1_Link: geometry collision mesh filename=package://jetcobot_description/meshes/LInk_1.stl; visual mesh filename=package://jetcobot_description/meshes/LInk_1.stl
- link 2_Link: geometry collision mesh filename=package://jetcobot_description/meshes/LInk_2.stl; visual mesh filename=package://jetcobot_description/meshes/LInk_2.stl
- link 3_Link: geometry collision mesh filename=package://jetcobot_description/meshes/LInk_3.stl; visual mesh filename=package://jetcobot_description/meshes/LInk_3.stl
- link 4_Link: geometry collision mesh filename=package://jetcobot_description/meshes/LInk_4.stl; visual mesh filename=package://jetcobot_description/meshes/LInk_4.stl
- link 5_Link: geometry collision mesh filename=package://jetcobot_description/meshes/LInk_5.stl; visual mesh filename=package://jetcobot_description/meshes/LInk_5.stl
- link 6_Link: geometry collision mesh filename=package://jetcobot_description/meshes/LInk_6.stl; visual mesh filename=package://jetcobot_description/meshes/LInk_6.stl
Joints:
- joint 2_Joint: axis -0.000732413960501075 -0.999999731784859 0 -> 0 -1 0
- joint 3_Joint: axis 0.000732413960503172 -0.999999731784859 0 -> 0 -1 0
- joint 4_Joint: axis 0.000732413960503879 -0.999999731784859 0 -> 0 -1 0
- joint 5_Joint: axis -1.63178762811156E-05 0 0.999999999866863 -> 0 0 1
- joint 6_Joint: axis 0.999999508360072 0.00099147029270504 -1.63178800449753E-05 -> 1 0 0

File: jetcobot_description/urdf/jetcobot_display_fixed.urdf (robot description, URDF)
Before this commit: robot jetcobot, 12 links, 11 joints
Links:
- removed link 1_Link
- removed link 2_Link
- removed link 3_Link
- removed link 4_Link
- removed link 5_Link
- removed link 6_Link
- removed link TCP
- removed link gripper_link
- removed link jetcocam
- removed link ov3360
- added link camera_link, mass 0.0173158610148997; collision mesh filename=package://jetcobot_description/meshes/camera_Link.STL; visual mesh filename=package://jetcobot_description/meshes/camera_Link.STL
- added link gripper_base; collision mesh filename=package://jetcobot_description/meshes/gripper_base.dae; visual mesh filename=package://jetcobot_description/meshes/gripper_base.dae
- added link gripper_left1; collision mesh filename=package://jetcobot_description/meshes/gripper_left1.dae; visual mesh filename=package://jetcobot_description/meshes/gripper_left1.dae
- added link gripper_left2; collision mesh filename=package://jetcobot_description/meshes/gripper_left2.dae; visual mesh filename=package://jetcobot_description/meshes/gripper_left2.dae
- added link gripper_left3; collision mesh filename=package://jetcobot_description/meshes/gripper_left3.dae; visual mesh filename=package://jetcobot_description/meshes/gripper_left3.dae
- added link gripper_right1; collision mesh filename=package://jetcobot_description/meshes/gripper_right1.dae; visual mesh filename=package://jetcobot_description/meshes/gripper_right1.dae
- added link gripper_right2; collision mesh filename=package://jetcobot_description/meshes/gripper_right2.dae; visual mesh filename=package://jetcobot_description/meshes/gripper_right2.dae
- added link gripper_right3; collision mesh filename=package://jetcobot_description/meshes/gripper_right3.dae; visual mesh filename=package://jetcobot_description/meshes/gripper_right3.dae
- added link link_1, mass 0.0362552727733653; collision mesh filename=package://jetcobot_description/meshes/Link_1.STL; visual mesh filename=package://jetcobot_description/meshes/Link_1.STL
- added link link_2, mass 0.0668252611526333; collision mesh filename=package://jetcobot_description/meshes/Link_2.STL; visual mesh filename=package://jetcobot_description/meshes/Link_2.STL
- added link link_3, mass 0.0533199813011819; collision mesh filename=package://jetcobot_description/meshes/Link_3.STL; visual mesh filename=package://jetcobot_description/meshes/Link_3.STL
- added link link_4, mass 0.0240531902650696; collision mesh filename=package://jetcobot_description/meshes/Link_4.STL; visual mesh filename=package://jetcobot_description/meshes/Link_4.STL
- added link link_5, mass 0.0314577601971656; collision mesh filename=package://jetcobot_description/meshes/Link_5.STL; visual mesh filename=package://jetcobot_description/meshes/Link_5.STL
- added link link_6, mass 0.00770526463879312; collision mesh filename=package://jetcobot_description/meshes/Link_6.STL; visual mesh filename=package://jetcobot_description/meshes/Link_6.STL
Joints:
- removed joint 1_Joint
- removed joint 2_Joint
- removed joint 3_Joint
- removed joint 4_Joint
- removed joint 5_Joint
- removed joint 6_Joint
- removed joint TCP_joint
- removed joint camera_joint
- removed joint gripper_Joint
- removed joint ov3360_joint
- added joint camera_Joint: type fixed, parent link_6, child camera_link, origin xyz=0.033 0 0.035 rpy=0 0 0, axis 0 0 0
- added joint gripper_base_to_gripper_left2: type revolute, parent gripper_base, child gripper_left2, origin xyz=-0.005 0.0195 0 rpy=0 0 0, axis 0 0 1, limit lower=-0.8 upper=0.5 effort=1000.0 velocity=0, mimic joint=gripper_controller multiplier=1.0 offset=0
- added joint gripper_base_to_gripper_right2: type revolute, parent gripper_base, child gripper_right2, origin xyz=0.005 0.0195 0 rpy=0 0 0, axis 0 0 1, limit lower=-0.5 upper=0.8 effort=1000.0 velocity=0, mimic joint=gripper_controller multiplier=-1.0 offset=0
- added joint gripper_base_to_gripper_right3: type revolute, parent gripper_base, child gripper_right3, origin xyz=0.012 -0.0025 0 rpy=0 0 0, axis 0 0 1, limit lower=-0.15 upper=0.7 effort=1000.0 velocity=0, mimic joint=gripper_controller multiplier=-1.0 offset=0
- added joint gripper_controller: type revolute, parent gripper_base, child gripper_left3, origin xyz=-0.012 -0.0025 0 rpy=0 0 0, axis 0 0 1, limit lower=-0.7 upper=0.15 effort=1000.0 velocity=0
- added joint gripper_left3_to_gripper_left1: type revolute, parent gripper_left3, child gripper_left1, origin xyz=-0.027 0.016 0 rpy=0 0 0, axis 0 0 1, limit lower=-0.5 upper=0.5 effort=1000.0 velocity=0, mimic joint=gripper_controller multiplier=-1.0 offset=0
- added joint gripper_right3_to_gripper_right1: type revolute, parent gripper_right3, child gripper_right1, origin xyz=0.027 0.016 0 rpy=0 0 0, axis 0 0 1, limit lower=-0.5 upper=0.5 effort=1000.0 velocity=0, mimic joint=gripper_controller multiplier=1.0 offset=0
- added joint joint_1: type revolute, parent base_link, child link_1, origin xyz=0 0 0.074520000000001 rpy=0 0 0, axis 0 0 1, limit lower=-2.87 upper=2.87 effort=0 velocity=0
- added joint joint_2: type revolute, parent link_1, child link_2, origin xyz=-2.56344886174708E-05 -0.0349999906124702 0.06 rpy=0 0 0, axis -0.000732413960501075 -0.999999731784859 0, limit lower=-2.87 upper=2.87 effort=0 velocity=0
- added joint joint_3: type revolute, parent link_2, child link_3, origin xyz=0 0.00678999562722426 0.109999999944807 rpy=0 0 0, axis 0.000732413960503172 -0.999999731784859 0, limit lower=-2.87 upper=2.87 effort=0 velocity=0
- added joint joint_4: type revolute, parent link_3, child link_4, origin xyz=0 -0.00134543437627838 0.0959999996761873 rpy=0 0 0, axis 0.000732413960503879 -0.999999731784859 0, limit lower=-2.87 upper=2.87 effort=0 velocity=0
- added joint joint_5: type revolute, parent link_4, child link_5, origin xyz=-2.51335035583085E-05 -0.0335399905878049 0.0348292449246146 rpy=0 0 0, axis -1.63178762811156E-05 0 0.999999999866863, limit lower=-2.87 upper=2.87 effort=0 velocity=0
- added joint joint_6: type revolute, parent link_5, child link_6, origin xyz=0.0319651869150594 -2.83148869312522E-05 0.03992044757551 rpy=0.785398 0 0, axis 0.999999508360072 0.00099147029270504 -1.63178800449753E-05, limit lower=-3.05 upper=3.05 effort=0 velocity=0
- added joint link_6_to_gripper_base: type fixed, parent link_6, child gripper_base, origin xyz=0.045 0 0 rpy=3.141592653589793 0 1.570796326794897
