Commit message: Edit loadpoint, Add new SCAN_PINK at picker_gui

File: pinky_description/urdf/robot_core.xacro (robot description, xacro)
@@ -72,5 +72,5 @@
         </xacro:inertial_sphere>
     </link>
-    <joint name="left_wheel_joint" type="continuous">
+    <joint name="left_wheel_joint" type="fixed">
         <parent link="${ns_prefix}base_link"/>
         <child link="${ns_prefix}left_wheel"/>
@@ -95,5 +95,5 @@
         </xacro:inertial_cylinder>
     </link>
-    <joint name="right_wheel_joint" type="continuous">
+    <joint name="right_wheel_joint" type="fixed">
         <parent link="${ns_prefix}base_link"/>
         <child link="${ns_prefix}right_wheel"/>
